File: PI_Shield.brd (EAGLE design)
At the start: 72.4 x 72.4 mm, 74 parts, among them J10 T2I, J11 T2I, J12 T2I, J13 DF13-4P-1.25DSA, J14 DF13-4P-1.25DSA, J15 DF13-4P-1.25DSA, J16 T2I5P, Q1 220mA/50V/3.5Ω, Q2 220mA/50V/3.5Ω, Q3 220mA/50V/3.5Ω, Q4 220mA/50V/3.5Ω, Q5 2.5A/30V/105mΩ, U1 MAX1136EUA-T, U2 AZ1117EH-3.3TRG1, Y1 ECS-80-S-4X

Commit message: Started routing
Parts:
- moved R22 5.21 mm to (32.6, 7.62), flipped to the top
- moved R25 3.44 mm to (41.4, 7.75)
- moved Q2 3.04 mm to (37.2, 8.76), turned to 0 degrees
- moved R23 2.85 mm to (23.8, 6.99), flipped to the bottom, turned to 90 degrees
- moved R17 2.62 mm to (29.4, 17.2)
- moved D4 2.35 mm to (27.1, 17.3)
- moved R24 1.91 mm to (26.2, 9.02)
- moved C9 1.86 mm to (20.1, 23.1)
- moved U$3 1.78 mm to (50.2, 3.68)
- moved U1 1.66 mm to (21.4, 19.8)
- moved C8 1.31 mm to (22.3, 16.9), flipped to the bottom, turned to 180 degrees
- moved C7 1.15 mm to (4.45, 8.89)
- moved R13 1.02 mm to (35.2, 12.2)
- moved R14 0.99 mm to (35.2, 16.1)
- moved U$6 0.98 mm to (38.6, 4.93)
Routing:
- net 5V: track 0.00 -> 88.1 mm, vias 0 -> 7
- net 5V_RAW: track 0.00 -> 52.8 mm
- net PI_POWER: track 0.00 -> 39.6 mm
- net SDA_ADC: track 0.00 -> 22.4 mm
- net SCL_ADC: track 0.00 -> 20.9 mm
- net AMP_OUT: track 0.00 -> 15.0 mm, vias 0 -> 1
- net AIN2: track 0.00 -> 13.7 mm, vias 0 -> 1
- net 3V3: track 0.00 -> 11.4 mm
- net N$13: track 0.00 -> 10.9 mm
- net OCD: track 0.00 -> 9.11 mm, vias 0 -> 1
- net !AMP_RESET: track 0.00 -> 6.71 mm, vias 0 -> 1
- net !AMP_FAULT: track 0.00 -> 5.31 mm, vias 0 -> 1
- net N$3: track 0.00 -> 5.07 mm, vias 0 -> 1
- net N$2: track 0.00 -> 4.82 mm, vias 0 -> 1
- net N$10: track 0.00 -> 4.25 mm, vias 0 -> 1
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- added copper zone on layer 1, net 5V
- added copper zone on layer 1, net 5V_RAW
- added copper zone on layer 1, net GND
- added copper zone on layer 16, net GND

Commit message: routed some
Parts:
- moved C5 13.2 mm to (30.7, 65.0), flipped to the bottom, turned to 270 degrees
- moved R5 11.2 mm to (31.8, 69.7), turned to 90 degrees
- moved J4 10.9 mm to (34.2, 57.9), turned to 270 degrees
- moved U$2 10.2 mm to (33.3, 67.2), turned to 180 degrees
- moved D2 9.44 mm to (34.5, 69.7)
- moved C13 8.45 mm to (42.2, 29.6), turned to 270 degrees
- moved J1 8.40 mm to (66.9, 34.5), turned to 90 degrees
- moved J12 8.13 mm to (5.21, 41.5)
- moved R6 7.78 mm to (37.1, 64.1), flipped to the top, turned to 0 degrees
- moved Q4 7.73 mm to (37.7, 69.7), turned to 90 degrees
- moved R3 6.22 mm to (37.5, 61.6), flipped to the bottom
- moved R7 4.47 mm to (37.1, 65.8), flipped to the top, turned to 180 degrees
- moved R4 4.06 mm to (37.3, 69.6), flipped to the bottom, turned to 90 degrees
- moved R10 3.72 mm to (20.6, 40.0), turned to 180 degrees
- moved C7 3.06 mm to (3.53, 11.8), turned to 90 degrees
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Connections:
- net N$9 renamed RESET_MID
- removed net G_INT: U$4.GI1, U$8.22
- net DI1: now also J12.2; no longer J12.3
- net DI2: now also J12.3; no longer J12.2
- net IMU_INT: now also U$4.GI1
- net INT: now also U$8.37; no longer U$8.35
- net RX: now also J8.2; no longer J8.3
- net RX0_INT: now also U$8.35; no longer U$8.37
- net TX: now also J8.3; no longer J8.2
Routing:
- net 3V3: track 11.4 -> 187.7 mm, vias 0 -> 2
- net 5V: track 88.1 -> 154.5 mm, vias 7 -> 8
- net A_INT: track 0.00 -> 53.3 mm, vias 0 -> 1
- net IMU_INT: track 0.00 -> 48.1 mm, vias 0 -> 1
- net PWM: track 0.00 -> 45.3 mm
- net !AMP_RESET: track 6.71 -> 42.0 mm
- net IMU_RESET: track 0.00 -> 27.9 mm
- net CS: track 0.00 -> 21.2 mm, vias 0 -> 1
- net MOSI: track 0.00 -> 20.2 mm, vias 0 -> 1
- net MISO: track 0.00 -> 18.3 mm
- net CLK: track 0.00 -> 14.8 mm
- net PI_POWER: track 39.6 -> 25.6 mm
- net CAN_RESET: track 0.00 -> 13.6 mm
- net RESET_MID: track 0.00 -> 12.2 mm, vias 0 -> 1
- net N$1: track 0.00 -> 11.9 mm
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- added copper zone on layer 1, net PI_POWER
